Commit message: update serial_drive + arduino

File: description/battery.xacro (robot description, xacro)
@@ -1,55 +1,41 @@
 <?xml version="1.0"?>
 <robot xmlns:xacro="http://www.ros.org/wiki/xacro" >
-  <!-- ********************* The Battery (Power System) SETUP *********************************  -->
-  <!-- See https://docs.ros.org/en/jazzy/p/battery_state_broadcaster/
-           https://github.com/gazebosim/ros_gz/blob/jazzy/ros_gz_sim_demos/README.md#battery
-           /opt/ros/jazzy/opt/gz_sim_vendor/share/gz/gz-sim8/worlds/linear_battery_demo.sdf
-           /opt/ros/jazzy/share/ros_gz_sim_demos
-           https://gazebosim.org/api/sim/7/battery.html
-      Note: This is generic SIM battery. Copy to robots/<robot_model>/description/. and customize.
-            Modify robot.urdf.xacro to include the customized version.
-      parameters: open_circuit_voltage
-                  battery_capacity
-  -->
-  <ros2_control name="BatteryState" type="diffdrive_arduino/DiffDriveArduino">
-    <sensor name="main_battery">
-        <!-- See diffdrive_arduino/src/diffdrive_arduino.cpp export_state_interfaces()-->
-        <state_interface name="voltage"/>
-        <state_interface name="temperature"/>
-        <state_interface name="current"/>
-        <state_interface name="charge"/>
-        <state_interface name="capacity"/>
-        <state_interface name="percentage"/>
-        <state_interface name="power_supply_status"/>
-        <state_interface name="power_supply_health"/>
-        <state_interface name="present"/>
-   </sensor>
-  </ros2_control>
+  <xacro:unless value="$(arg sim_mode)">
+      <ros2_control name="BatteryState" type="sensor">
+        <hardware>
+            <plugin>diffdrive_arduino/DiffDriveArduino</plugin>
+            <param name="device">/dev/ttyACM0</param>
+            <param name="baud_rate">115200</param>
+            <param name="timeout">1000</param>
+        </hardware>
+        <sensor name="main_battery">
+            <state_interface name="voltage"/>
+            <state_interface name="temperature"/>
+            <state_interface name="current"/>
+            <state_interface name="charge"/>
+            <state_interface name="capacity"/>
+            <state_interface name="percentage"/>
+            <state_interface name="power_supply_status"/>
+            <state_interface name="power_supply_health"/>
+            <state_interface name="present"/>
+       </sensor>
+      </ros2_control>
+  </xacro:unless>
   <gazebo>
     <plugin name="gz::sim::systems::LinearBatteryPlugin" filename="gz-sim-linearbatteryplugin-system">
-      <!--Li-ion battery spec from LIR18650 datasheet-->
       <battery_name>lithium_battery</battery_name>
       <voltage>${open_circuit_voltage}</voltage>
       <open_circuit_voltage_constant_coef>${open_circuit_voltage}</open_circuit_voltage_constant_coef>
       <open_circuit_voltage_linear_coef>-2.0</open_circuit_voltage_linear_coef>
-      <initial_charge>${battery_capacity * 0.9}</initial_charge>
+      <initial_charge>${battery_capacity}</initial_charge>
       <capacity>${battery_capacity}</capacity>
       <resistance>0.07</resistance>
+      <smooth_current_tau>2.0</smooth_current_tau>
       <power_load>6.6</power_load>
-      <smooth_current_tau>2.0</smooth_current_tau>
-      <!-- if "fix_issue_225" is true, percentage is reported in 1..100 range which is wrong.
-               see https://github.com/gazebosim/gz-sim/issues/225 -->
-      <fix_issue_225>false</fix_issue_225>
-      <!-- https://github.com/gazebosim/gz-sim/pull/2696 -->
-      <invert_current_sign>true</invert_current_sign>
+      <soc_threshold>0.51</soc_threshold>
+      <fix_issue_225>false</fix_issue_225> <invert_current_sign>true</invert_current_sign>
       <enable_recharge>true</enable_recharge>
-      <!-- charging I = c / t, discharging I = P / V,
-        charging I should be > discharging I -->
+      <recharge_by_topic>true</recharge_by_topic>
       <charging_time>3.0</charging_time>
-      <!-- Consumer-specific -->
-      <soc_threshold>0.51</soc_threshold>
-      <power_load>2.1</power_load>
-      <recharge_by_topic>true</recharge_by_topic>
-      <start_on_motion>true</start_on_motion>
     </plugin>
   </gazebo>

File: description/camera.xacro (robot description, xacro)
@@ -1,86 +1,92 @@
 <?xml version="1.0"?>
 <robot xmlns:xacro="http://www.ros.org/wiki/xacro" >
-    <!-- parameters: camera_offset_x
-                     camera_offset_z -->
-    <joint name="camera_joint" type="fixed">
-        <parent link="chassis_link"/>
-        <child link="camera_link"/>
-        <origin xyz="${camera_offset_x} 0 ${camera_offset_z}" rpy="0 0.18 0"/>
+    <!-- Raspberry Pi Camera v2.1 approximate body dimensions. -->
+    <xacro:property name="pi_cam_board_x" value="0.025"/>
+    <xacro:property name="pi_cam_board_y" value="0.024"/>
+    <xacro:property name="pi_cam_board_z" value="0.002"/>
+    <xacro:property name="pi_cam_lens_radius" value="0.0045"/>
+    <xacro:property name="pi_cam_lens_length" value="0.006"/>
+    <xacro:property name="pi_cam_support_radius" value="0.004"/>
+    <xacro:property name="pi_cam_support_length" value="0.030"/>
+    <joint name="camera_joint" type="revolute">
+      <parent link="chassis"/>
+         <child link="camera_link"/>
+         <origin xyz="${camera_offset_x} 0 ${camera_offset_z}" rpy="0 0 0"/>
+         <axis xyz="0 1 0"/>
+         <limit lower="-0.70" upper="0.35" effort="2.0" velocity="1.0"/>
+         <dynamics damping="0.2" friction="0.05"/>
     </joint>
     <link name="camera_link">
         <visual>
             <geometry>
-                <box size="0.010 0.03 0.03"/>
+                <box size="${pi_cam_board_x} ${pi_cam_board_y} ${pi_cam_board_z}"/>
             </geometry>
-            <material name="sensor_blue"/>
+            <material name="blue">
+                 <color rgba="0.2 0.2 1 1"/>
+            </material>
         </visual>
         <visual>
-            <origin xyz="0 0 -0.05"/>
+            <origin xyz="${pi_cam_board_x/2 + pi_cam_lens_length/2} 0 0"/>
             <geometry>
-                <cylinder radius="0.002" length="0.1"/>
+                <cylinder radius="${pi_cam_lens_radius}" length="${pi_cam_lens_length}"/>
             </geometry>
-            <material name="sensor_blue"/>
+            <material name="black"/>
         </visual>
+        <visual>
+            <origin xyz="0 0 ${-(pi_cam_support_length/2 + pi_cam_board_z/2)}"/>
+            <geometry>
+                <cylinder radius="${pi_cam_support_radius}" length="${pi_cam_support_length}"/>
+            </geometry>
+            <material name="grey"/>
+        </visual>
+        <collision>
+            <geometry>
+                <box size="${pi_cam_board_x} ${pi_cam_board_y} ${pi_cam_board_z}"/>
+            </geometry>
+        </collision>
+        <collision>
+            <origin xyz="${pi_cam_board_x/2 + pi_cam_lens_length/2} 0 0"/>
+            <geometry>
+                <cylinder radius="${pi_cam_lens_radius}" length="${pi_cam_lens_length}"/>
+            </geometry>
+        </collision>
+        <collision>
+            <origin xyz="0 0 ${-(pi_cam_support_length/2 + pi_cam_board_z/2)}"/>
+            <geometry>
+                <cylinder radius="${pi_cam_support_radius}" length="${pi_cam_support_length}"/>
+            </geometry>
+        </collision>
+        <xacro:inertial_box mass="0.01" x="${pi_cam_board_x}" y="${pi_cam_board_y}" z="${pi_cam_board_z}">
+            <origin xyz="0 0 0" rpy="0 0 0"/>
+        </xacro:inertial_box>
     </link>
     <joint name="camera_optical_joint" type="fixed">
         <parent link="camera_link"/>
         <child link="camera_link_optical"/>
-        <origin xyz="0 0 0" rpy="0 0 0"/>
+        <origin xyz="0 0 0" rpy="${-pi/2} 0 ${-pi/2}"/>
     </joint>
     <link name="camera_link_optical">
     </link>
-    <!-- gz model -m dragger -s rgb_camera -->
-	  <gazebo reference="camera_link_optical">
+    <gazebo reference="camera_link">
         <sensor name='rgb_camera' type='camera'>
-          <pose>0 0 0 0 0 0</pose>
-		      <always_on>true</always_on>
-          <topic>gz_camera</topic>
-          <!-- future Gazebo versions might require "<frame_id>" here. Must reference an actual link in .xacro -->
-          <!-- see <optical_frame_id> below     <gz_frame_id>camera_link_optical</gz_frame_id> -->
-          <update_rate>10</update_rate>
-          <visualize>true</visualize>
-          <enable_metrics>false</enable_metrics>
-          <camera name='__default__'>
             <pose>0 0 0 0 0 0</pose>
-            <horizontal_fov>1.047</horizontal_fov>
-            <image>
-              <width>320</width>
-              <height>240</height>
-              <format>RGB_INT8</format>
-              <anti_aliasing>4</anti_aliasing>
-            </image>
-            <camera_info_topic>gz_camera_info</camera_info_topic>
-            <trigger_topic></trigger_topic>
-            <triggered>false</triggered>
-            <clip>
-              <near>0.10000000000000001</near>
-              <far>100</far>
-            </clip>
-            <save enabled='false'>
-              <path>__default__</path>
-            </save>
-            <visibility_mask>4294967295</visibility_mask>
-            <noise>
-              <type>none</type>
-              <mean>0</mean>
-              <stddev>0</stddev>
-            </noise>
-            <distortion>
-              <k1>0</k1>
-              <k2>0</k2>
-              <k3>0</k3>
-              <p1>0</p1>
-              <p2>0</p2>
-              <center>0.5 0.5</center>
-            </distortion>
-            <lens>
-              <type>stereographic</type>
-              <scale_to_hfov>true</scale_to_hfov>
-              <cutoff_angle>${pi/2}</cutoff_angle>
-              <env_texture_size>256</env_texture_size>
-            </lens>
-            <optical_frame_id>camera_link_optical</optical_frame_id>
-          </camera>
-        </sensor>
+            <visualize>true</visualize>
+            <update_rate>10</update_rate>
+            <topic>camera/image_raw</topic>
+            <gz_frame_id>camera_link_optical</gz_frame_id>
+            <camera name='__default__'>
+                <horizontal_fov>1.089</horizontal_fov>
+                <image>
+                    <width>640</width>
+                    <height>480</height>
+                    <format>R8G8B8</format>
+                </image>
+                <clip>
+                    <near>0.05</near>
+                    <far>8.0</far>
+                </clip>
+                <optical_frame_id>camera_link_optical</optical_frame_id>
+            </camera>
+            </sensor>
     </gazebo>
 </robot>

File: description/common_properties.xacro (robot description, xacro)
@@ -1,5 +1,5 @@
 <?xml version="1.0" ?>
-<robot name="xacro_properties"
-  xmlns:xacro="http://ros.org/wiki/xacro">
+<robot name="xacro_properties" xmlns:xacro="http://ros.org/wiki/xacro">
+    <xacro:arg name="sim_mode" default="false"/>
     <material name="white">
         <color rgba="1 1 1 1" />
@@ -10,4 +10,7 @@
     <material name="red">
         <color rgba="1 0 0 1"/>
+    </material>
+    <material name="orange">
+        <color rgba="1 0.3 0.1 1"/>
     </material>
     <material name="green">
@@ -30,6 +33,5 @@
     </material>
     <material name="body_color">
-        <color rgba="0.6 0.5 0.2 0.85"/>
-    </material>
+        <color rgba="0.1 0.1 0.1 1"/> </material>
     <material name="port_red">
         <color rgba="1 0.2 0.2 1"/>
@@ -38,4 +40,3 @@
         <color rgba="0.2 1 0.2 1"/>
     </material>
-    <xacro:arg name="sim_mode" default="false"/>
 </robot>

File: description/imu.xacro (robot description, xacro)
@@ -1,13 +1,7 @@
 <?xml version="1.0"?>
 <robot xmlns:xacro="http://www.ros.org/wiki/xacro" >
-    <!-- *********************** IMU SETUP *********************************  -->
-    <!-- Each sensor must be attached to a link.                              -->
-    <!-- parameters: imu_offset_x
-                     imu_offset_z
-                     imu_visual_size -->
     <joint name="imu_joint" type="fixed">
-        <parent link="chassis_link"/>
+        <parent link="chassis"/>
         <child link="imu_link"/>
-        <!-- we want to place IMU closely between the wheels, at center mass -->
         <origin xyz="${imu_offset_x} 0 ${imu_offset_z}" rpy="0 0 0"/>
     </joint>
@@ -19,14 +13,18 @@
             <material name="sensor_blue"/>
         </visual>
+        <collision>
+            <geometry>
+                <box size="${imu_visual_size} ${imu_visual_size} ${imu_visual_size}"/>
+            </geometry>
+        </collision>
+        <xacro:inertial_box mass="0.01" x="${imu_visual_size}" y="${imu_visual_size}" z="${imu_visual_size}">
+            <origin xyz="0 0 0" rpy="0 0 0"/>
+        </xacro:inertial_box>
     </link>
-    <!-- gz model -m dragger -s imu_link -->
     <gazebo reference="imu_link">
-        <!-- IMU sensor, with "enable_orientation" publishes /imu/data, without - /imu/data_raw
-             See https://github.com/CCNYRoboticsLab/imu_tools -->
         <sensor name="imu_link" type="imu">
         <pose>0 0 0 0 0 0</pose>
         <always_on>1</always_on>
         <topic>gz_imu/data</topic>
-        <!-- future Gazebo versions might require "<frame_id>" here. Must reference an actual link in .xacro -->
         <gz_frame_id>imu_link</gz_frame_id>
         <frame_id>imu_link</frame_id>
@@ -35,6 +33,5 @@
                 <orientation_reference_frame>
                   <localization>ENU</localization>
-                  <!-- custom_rpy parent_frame='world'>1.570795 0 0</custom_rpy -->
-                </orientation_reference_frame>
+                  </orientation_reference_frame>
                 <enable_orientation>1</enable_orientation>
                 <angular_velocity>
@@ -110,5 +107,4 @@
             </imu>
         </sensor>
-        <!-- Magnetometer sharing the IMU link, taking magnetic field from "gz::sim::systems::Magnetometer" Gazebo plugin -->
         <sensor name="magnetometer" type="magnetometer">
           <pose>0 0 0 0 0 0</pose>
@@ -117,5 +113,4 @@
           <visualize>true</visualize>
           <topic>gz_magnetometer/data</topic>
-          <!-- future Gazebo versions might require "<frame_id>" here. Must reference an actual link in .xacro -->
           <gz_frame_id>imu_link</gz_frame_id>
           <frame_id>imu_link</frame_id>

File: description/lidar.xacro (robot description, xacro)
@@ -1,63 +1,57 @@
 <?xml version="1.0"?>
 <robot xmlns:xacro="http://www.ros.org/wiki/xacro" >
-    <!-- ********************* LIDAR SETUP *********************************  -->
-    <!-- Each sensor must be attached to a link.                              -->
-    <xacro:arg name="lidar_offset_x" default="0"/>
-    <xacro:arg name="lidar_offset_z" default="0"/>
+    <xacro:arg name="lidar_offset_x" default="-0.08"/>
+    <xacro:arg name="lidar_offset_y" default="0.0"/>
+    <!-- Relative height above chassis top (meters), to LiDAR center. -->
+    <xacro:arg name="lidar_offset_z" default="0.0275"/>
     <xacro:arg name="lidar_min_angle" default="-3.14159"/>
     <xacro:arg name="lidar_max_angle" default="3.14159"/>
-    <xacro:arg name="lidar_pedestal_height" default="0.003"/>
-    <xacro:property name="_lidar_pedestal_height" value="$(arg lidar_pedestal_height)"/>
+    <xacro:property name="lidar_offset_x_val" value="$(arg lidar_offset_x)"/>
+    <xacro:property name="lidar_offset_y_val" value="$(arg lidar_offset_y)"/>
+    <xacro:property name="lidar_offset_z_val" value="$(arg lidar_offset_z)"/>
+    <!-- RPLidar A1 physical envelope from provided dimensions: 70mm diameter, ~55mm height. -->
+    <xacro:property name="lidar_body_radius" value="0.035"/>
+    <xacro:property name="lidar_body_height" value="0.055"/>
+    <xacro:property name="lidar_body_mass" value="0.17"/>
     <joint name="laser_joint" type="fixed">
-        <parent link="chassis_link"/>
+        <parent link="chassis"/>
         <child link="laser_frame"/>
-        <origin xyz="$(arg lidar_offset_x) 0 $(arg lidar_offset_z)" rpy="0 0 0"/>
+        <origin xyz="${lidar_offset_x_val} ${lidar_offset_y_val} ${chassis_height + lidar_offset_z_val}" rpy="0 0 0"/>
     </joint>
-    <!-- the name "laser_frame" should correspond to /scan topic header->frame_id as defined in *.launch.py -->
+    <gazebo reference="laser_joint">
+    <preserveFixedJoint>true</preserveFixedJoint>
+    </gazebo>
     <link name="laser_frame">
-        <visual name="lidar_visual_scanner">
+        <visual>
             <geometry>
-                <cylinder radius="0.03" length="0.02"/>
+                <cylinder radius="${lidar_body_radius}" length="${lidar_body_height}"/>
             </geometry>
-            <material name="sensor_blue"/>
-        </visual>
-        <visual name="lidar_visual_motor">
-            <origin xyz="0.03 0 -0.01"/>
-            <geometry>
-                <cylinder radius="0.012" length="0.01"/>
-            </geometry>
-            <material name="sensor_blue"/>
-        </visual>
-        <visual name="lidar_visual_base">
-            <origin xyz="0 0 -${_lidar_pedestal_height/2+0.01}"/>
-            <geometry>
-                <cylinder radius="0.02" length="${_lidar_pedestal_height}"/>
-            </geometry>
-            <material name="body_color"/>
+            <material name="blue"/>
         </visual>
         <collision>
             <geometry>
-                <cylinder radius="0.05" length="0.04"/>
+                <cylinder radius="${lidar_body_radius}" length="${lidar_body_height}"/>
             </geometry>
         </collision>
-        <xacro:inertial_cylinder mass="0.1" length="0.04" radius="0.05">
+        <xacro:inertial_cylinder mass="${lidar_body_mass}" length="${lidar_body_height}" radius="${lidar_body_radius}">
             <origin xyz="0 0 0" rpy="0 0 0"/>
         </xacro:inertial_cylinder>
     </link>
-    <!-- gz model -m dragger -s laser_frame -->
     <gazebo reference="laser_frame">
-        <!-- name must be "laser_frame", specifically for lasers. Must reference an actual link in .xacro -->
-        <sensor name='laser_frame' type='gpu_lidar'>
+        <material>Gazebo/Blue</material>
+    </gazebo>
+    <gazebo reference="laser_frame">
+        <sensor name='laser_sensor' type='gpu_lidar'>
           <pose>0 0 0 0 0 0</pose>
           <always_on>1</always_on>
-          <!-- 6 Hz for LD14 - see "frequency" in dual_ekf_navsat_parameters.yaml -->
-          <update_rate>6</update_rate>
-          <topic>gz_scan</topic>
-          <!-- future Gazebo versions might require "<frame_id>" here. Must reference an actual link in .xacro -->
+          <!-- Stable sim profile for mapping: improve temporal consistency while keeping load bounded. -->
+          <update_rate>10.0</update_rate>
+          <topic>/scan</topic>
           <gz_frame_id>laser_frame</gz_frame_id>
           <frame_id>laser_frame</frame_id>
-          <ray>
+          <visualize>false</visualize> <ray>
             <scan>
               <horizontal>
+                <!-- 360 samples/scan @ 8Hz ~= 2880 samples/sec (similar load, better temporal response). -->
                 <samples>360</samples>
                 <resolution>1</resolution>
@@ -65,23 +59,15 @@
                 <max_angle>$(arg lidar_max_angle)</max_angle>
               </horizontal>
-              <vertical>
-                <samples>1</samples>
-                <resolution>1</resolution>
-                <min_angle>0</min_angle>
-                <max_angle>0</max_angle>
-              </vertical>
             </scan>
             <range>
-              <min>0.3</min>
-              <max>12.0</max>
+              <min>0.15</min> <max>12.0</max>
               <resolution>0.01</resolution>
             </range>
             <noise>
               <type>gaussian</type>
-              <mean>0</mean>
-              <stddev>0.01</stddev>
+              <mean>0.0</mean>
+              <stddev>0.005</stddev>
             </noise>
           </ray>
-          <visualize>true</visualize>
         </sensor>
     </gazebo>
