Commit message: Initial upload of alpha_robot

File: description/arm.xacro (robot description, xacro)
@@ -1,54 +1,46 @@
 <?xml version="1.0"?>
 <robot xmlns:xacro="http://www.ros.org/wiki/xacro" >
-    <!-- Real hardware profile from provided kit sheet:
-         base plate ~9cm x 8.4cm, overall chain length target ~50.5cm. -->
-    <xacro:property name="arm_base_radius" value="0.032"/>
+    <!-- Real hardware profile: base plate ~9cm x 4cm. -->
+    <xacro:property name="arm_base_size_x" value="0.09"/>
+    <xacro:property name="arm_base_size_y" value="0.04"/>
     <xacro:property name="arm_base_length" value="0.030"/>
     <xacro:property name="arm_base_mass" value="0.20"/>
-    <xacro:property name="link_1_radius" value="0.022"/>
-    <xacro:property name="link_1_length" value="0.050"/>
+    <xacro:property name="link_1_radius" value="0.0175"/>
+    <xacro:property name="link_1_length" value="0.025"/>
     <xacro:property name="link_1_mass" value="0.10"/>
-    <xacro:property name="link_2_radius" value="0.020"/>
-    <xacro:property name="link_2_length" value="0.140"/>
+    <xacro:property name="link_2_radius" value="0.0175"/>
+    <xacro:property name="link_2_length" value="0.100"/>
     <xacro:property name="link_2_mass" value="0.15"/>
-    <xacro:property name="link_3_radius" value="0.018"/>
-    <xacro:property name="link_3_length" value="0.125"/>
+    <xacro:property name="link_3_radius" value="0.0175"/>
+    <xacro:property name="link_3_length" value="0.105"/>
     <xacro:property name="link_3_mass" value="0.13"/>
-    <xacro:property name="link_4_radius" value="0.016"/>
+    <xacro:property name="link_4_radius" value="0.0175"/>
     <xacro:property name="link_4_length" value="0.070"/>
     <xacro:property name="link_4_mass" value="0.08"/>
-    <xacro:property name="link_5_radius" value="0.016"/>
-    <xacro:property name="link_5_length" value="0.050"/>
+    <xacro:property name="link_5_radius" value="0.0175"/>
+    <xacro:property name="link_5_length" value="0.030"/>
     <xacro:property name="link_5_mass" value="0.06"/>
-    <xacro:property name="link_6_radius" value="0.022"/>
-    <xacro:property name="link_6_length" value="0.040"/>
+    <xacro:property name="link_6_radius" value="0.0175"/>
+    <xacro:property name="link_6_length" value="0.084"/>
     <xacro:property name="link_6_mass" value="0.05"/>
     <joint name="arm_base_joint" type="fixed">
         <parent link="chassis"/>
         <child link="arm_base_link"/>
-        <origin xyz="0.07 0 ${chassis_height}" rpy="0 0 0"/>
+        <!-- Arm base center is 7.5 cm from front; robot half-length is 14.65 cm. -->
+        <origin xyz="0.0715 0 ${chassis_height}" rpy="0 0 0"/>
     </joint>
     <link name="arm_base_link">
         <visual>
             <origin xyz="0 0 ${arm_base_length/2}"/>
-            <geometry><cylinder radius="${arm_base_radius}" length="${arm_base_length}"/></geometry>
+            <geometry><box size="${arm_base_size_x} ${arm_base_size_y} ${arm_base_length}"/></geometry>
             <material name="orange"><color rgba="1 0.3 0.1 1"/></material>
-        </visual>
-        <visual>
-            <origin xyz="0 0 0.002"/>
-            <geometry><box size="0.09 0.084 0.004"/></geometry>
-            <material name="grey"/>
         </visual>
         <collision>
             <origin xyz="0 0 ${arm_base_length/2}"/>
-            <geometry><cylinder radius="${arm_base_radius}" length="${arm_base_length}"/></geometry>
+            <geometry><box size="${arm_base_size_x} ${arm_base_size_y} ${arm_base_length}"/></geometry>
         </collision>
-        <collision>
-            <origin xyz="0 0 0.002"/>
-            <geometry><box size="0.09 0.084 0.004"/></geometry>
-        </collision>
-        <xacro:inertial_cylinder mass="${arm_base_mass}" length="${arm_base_length}" radius="${arm_base_radius}">
+        <xacro:inertial_box mass="${arm_base_mass}" x="${arm_base_size_x}" y="${arm_base_size_y}" z="${arm_base_length}">
             <origin xyz="0 0 ${arm_base_length/2}" rpy="0 0 0"/>
-        </xacro:inertial_cylinder>
+        </xacro:inertial_box>
     </link>
     <joint name="joint_1" type="revolute">

File: description/camera.xacro (robot description, xacro)
@@ -9,11 +9,8 @@
     <xacro:property name="pi_cam_support_radius" value="0.004"/>
     <xacro:property name="pi_cam_support_length" value="0.030"/>
-    <joint name="camera_joint" type="revolute">
+    <joint name="camera_joint" type="fixed">
       <parent link="chassis"/>
          <child link="camera_link"/>
          <origin xyz="${camera_offset_x} 0 ${camera_offset_z}" rpy="0 0 0"/>
-         <axis xyz="0 1 0"/>
-         <limit lower="-0.70" upper="0.35" effort="2.0" velocity="1.0"/>
-         <dynamics damping="0.2" friction="0.05"/>
     </joint>
     <link name="camera_link">

File: description/lidar.xacro (robot description, xacro)
@@ -1,8 +1,10 @@
 <?xml version="1.0"?>
 <robot xmlns:xacro="http://www.ros.org/wiki/xacro" >
-    <xacro:arg name="lidar_offset_x" default="-0.08"/>
+    <xacro:arg name="lidar_offset_x" default="-0.0885"/>
     <xacro:arg name="lidar_offset_y" default="0.0"/>
     <!-- Relative height above chassis top (meters), to LiDAR center. -->
     <xacro:arg name="lidar_offset_z" default="0.0275"/>
+    <!-- Yaw of the physical LiDAR mounting relative to the robot front. -->
+    <xacro:arg name="lidar_yaw" default="0.0"/>
     <xacro:arg name="lidar_min_angle" default="-3.14159"/>
     <xacro:arg name="lidar_max_angle" default="3.14159"/>
@@ -10,4 +12,5 @@
     <xacro:property name="lidar_offset_y_val" value="$(arg lidar_offset_y)"/>
     <xacro:property name="lidar_offset_z_val" value="$(arg lidar_offset_z)"/>
+    <xacro:property name="lidar_yaw_val" value="$(arg lidar_yaw)"/>
     <!-- RPLidar A1 physical envelope from provided dimensions: 70mm diameter, ~55mm height. -->
     <xacro:property name="lidar_body_radius" value="0.035"/>
@@ -17,5 +20,5 @@
         <parent link="chassis"/>
         <child link="laser_frame"/>
-        <origin xyz="${lidar_offset_x_val} ${lidar_offset_y_val} ${chassis_height + lidar_offset_z_val}" rpy="0 0 0"/>
+        <origin xyz="${lidar_offset_x_val} ${lidar_offset_y_val} ${chassis_height + lidar_offset_z_val}" rpy="0 0 ${lidar_yaw_val}"/>
     </joint>
     <gazebo reference="laser_joint">

File: description/robot.urdf.xacro (robot description, xacro)
@@ -3,4 +3,5 @@
     <xacro:arg name="use_ros2_control" default="true"/>
     <xacro:arg name="sim_mode" default="false"/>
+    <xacro:arg name="include_arm" default="false"/>
     <xacro:include filename="common_properties.xacro" />
     <xacro:include filename="robot_core.xacro" />
@@ -14,5 +15,7 @@
     <xacro:property name="camera_offset_z" value="${chassis_height + 0.032}"/>
     <xacro:include filename="camera.xacro" />
-    <xacro:include filename="arm.xacro" />
+    <xacro:if value="$(arg include_arm)">
+        <xacro:include filename="arm.xacro" />
+    </xacro:if>
     <xacro:include filename="ros2_control.xacro" />
 </robot>

File: description/robot_core.xacro (robot description, xacro)
@@ -2,15 +2,18 @@
 <robot xmlns:xacro="http://www.ros.org/wiki/xacro" >
     <xacro:include filename="inertial_macros.xacro" />
-    <!-- Real hardware body size: 32 cm x 27 cm (without tyres). -->
-    <xacro:property name="chassis_length" value="0.32"/>
-    <xacro:property name="chassis_width" value="0.27"/>
-    <!-- Body top target from ground is ~12.6 cm with current tyres. -->
-    <xacro:property name="chassis_height" value="0.0795"/>
+    <!-- Real hardware body size (base plate). -->
+    <xacro:property name="chassis_length" value="0.293"/>
+    <!-- Base plate width (no wheels). -->
+    <xacro:property name="chassis_width" value="0.22"/>
+    <!-- Top of base is ~0.21 m above ground. -->
+    <xacro:property name="chassis_height" value="0.1735"/>
     <xacro:property name="chassis_mass" value="3.0"/>
-    <xacro:property name="wheel_radius" value="0.0425"/>
-    <xacro:property name="wheel_thickness" value="0.04"/>
+    <xacro:property name="wheel_radius" value="0.0325"/>
+    <xacro:property name="wheel_thickness" value="0.027"/>
     <xacro:property name="wheel_mass" value="0.2"/>
+    <!-- Wheelbase 0.22 m -> half is 0.11 m. -->
     <xacro:property name="wheel_offset_x" value="0.11"/>
-    <xacro:property name="wheel_offset_y" value="${(chassis_width / 2.0) + (wheel_thickness / 2.0)}"/>
+    <!-- Wheel separation 0.236 m -> half is 0.118 m. -->
+    <xacro:property name="wheel_offset_y" value="0.118"/>
     <xacro:property name="chassis_ground_clearance" value="0.004"/>
     <link name="base_link"></link>

File: description/ros2_control.xacro (robot description, xacro)
@@ -50,12 +50,5 @@
             <state_interface name="position"/>
         </joint>
-        <joint name="camera_joint">
-            <command_interface name="position">
-                <param name="min">-0.70</param>
-                <param name="max">0.35</param>
-            </command_interface>
-            <state_interface name="position"/>
-            <state_interface name="velocity"/>
-        </joint>
+        <xacro:if value="$(arg include_arm)">
         <joint name="joint_1">
             <command_interface name="position">
@@ -106,4 +99,5 @@
             <state_interface name="velocity"/>
         </joint>
+        </xacro:if>
     </ros2_control>
     <gazebo>
